File: hardware/phaser.kicad_pcb (KiCad board)
At the start: 2 copper layers, 10 parts, among them IC1 STM32F042K4U6, IC2 MCP1700, P2 SWD_TC

Commit message: Parts and rough board outlines
Parts:
- added C10: 4u7, agg:0603, F.Cu at (111.7, 35.7)
- added C11: 100n, agg:0603, F.Cu at (95.9, 51.7)
- added C12: 100n, agg:0603, F.Cu at (28.3, 74.9)
- added C13: 100n, agg:0603, F.Cu at (112.8, 42.8)
- added C14: 100n, agg:0603, F.Cu at (99.8, 43.8)
- added C6: 4u7, agg:0603, F.Cu at (34.8, 74.4)
- added C7: 100n, agg:0603, F.Cu at (41.3, 74.9)
- added D1: RED, agg:SIL-254P-02, F.Cu at (102.2, 55.5)
- added D2: YELLOW, agg:SIL-254P-02, F.Cu at (94.7, 65.3)
- added D3: BLUE, agg:SIL-254P-02, F.Cu at (87.2, 71.6)
- added F1: 100mA TD, footprints:5x20_clip, F.Cu at (175.2, 139.3)
- added IC3: LMx93, agg:SOIC-8, F.Cu at (105.3, 27.9)
- added IC4: AD8541, agg:SOT-23-5, F.Cu at (82.2, 64.7)
- added IC5: STM32F042K4U6, agg:QFN-32-EP-ST, F.Cu at (78.6, 56.6)
- added J1: MICROUSB, agg:MICROUSB_MOLEX_47589-0001, F.Cu at (91.4, 44.8)
- added P1: L, agg:SIL-254P-01, F.Cu at (194.2, 117.3)
- added P3: COAX, agg:SMA-EDGE, F.Cu at (93.7, 36.1)
- added P4: SWD_TC, agg:TC2030-NL, F.Cu at (113.0, 27.1)
- added P5: N, agg:SIL-254P-01, F.Cu at (155.6, 118.5)
- added Q1: BSS138P, agg:SOT-23, F.Cu at (105.0, 35.9)
- added Q2: BSS138P, agg:SOT-23, F.Cu at (74.1, 71.2)
- added Q3: BSS138P, agg:SOT-23, F.Cu at (63.2, 73.6)
- added R1: 1k8, agg:0603, F.Cu at (94.9, 60.5)
- added R10: 68, agg:0603, F.Cu at (106.3, 46.5)
- added R11: 68, agg:0603, F.Cu at (112.8, 39.0)
- added R12: 10k, agg:0603, F.Cu at (102.4, 50.7)
- added R2: 10k, agg:0603, F.Cu at (106.3, 43.3)
- added R3: 45k, agg:0603, F.Cu at (80.9, 69.8)
- added R4: 10k, agg:0603, F.Cu at (95.5, 55.3)
- added R5: 50k, agg:0603, F.Cu at (88.4, 60.5)
- added R6: 10k, agg:0603, F.Cu at (99.8, 47.4)
- added R7: 10k, agg:0603, F.Cu at (88.4, 63.6)
- added R8: 10k, agg:0603, F.Cu at (80.9, 72.9)
- added R9: 68, agg:0603, F.Cu at (106.3, 40.6)
- added SW1: SW, agg:SIL-254P-02, F.Cu at (112.6, 48.0)
- added SW2: CLK_SRC, agg:SIL-254P-03, F.Cu at (74.8, 64.5)
- added T1: 230/6+6 1VA, footprints:VB1.0-2-6, F.Cu at (175.0, 88.2)
- added U1: VTX-214-003-105, footprints:VTX214, F.Cu at (175.1, 119.6)
- added U2: FOX924B-20.000, footprints:FOX924, F.Cu at (57.3, 60.7)
- C1: value 1u -> 0.1uF/275V/X2; footprint agg:0603 -> footprints:ECQU2A104ML
- C2: value 10n -> 1u
- C4, C5: value 100n -> 1u
- C9: value 1u -> 10n
- IC1: value STM32F042K4U6 -> MCP1700; footprint agg:QFN-32-EP-ST -> agg:SOT-23
- IC2: value MCP1700 -> BQ24232HA; footprint agg:SOT-23 -> agg:QFN-16-EP-TI
- P2: value SWD_TC -> BATT; footprint agg:TC2030-NL -> footprints:JST-PH-2
- moved IC2 102.3 mm to (55.0, 72.4)
- moved C9 95.1 mm to (112.5, 32.5), turned to 0 degrees
- moved P2 91.1 mm to (67.3, 66.8)
- moved C8 88.4 mm to (89.4, 50.8), turned to 0 degrees
- moved C5 80.9 mm to (70.0, 75.9), turned to 0 degrees
- moved C4 72.3 mm to (99.8, 40.6), turned to 0 degrees
- moved IC1 71.9 mm to (88.7, 55.5)
- moved C2 67.4 mm to (76.5, 75.9), turned to 0 degrees
- moved C1 60.1 mm to (75.0, 115.0), turned to 0 degrees
- moved C3 58.9 mm to (88.4, 66.8), turned to 0 degrees
Connections:
- C1 pad 1: +3V3 -> /L
- C1 pad 2: GND -> /N
- C2 pad 1: +3V3 -> Net-(C2-Pad1)
- C3 pad 1: +3V3 -> Net-(C3-Pad1)
- C4 pad 1: +3V3 -> Net-(C3-Pad1)
- C8 pad 1: +5V -> +3V3
- IC1 pad 1: +3V3 -> GND
- IC1 pad 2: (no net) -> +3V3
- IC1 pad 3: (no net) -> Net-(C3-Pad1)
- IC2 pad 1: GND -> Net-(IC2-Pad1)
- IC2 pad 2: +3V3 -> Net-(C6-Pad1)
- IC2 pad 3: +5V -> Net-(C6-Pad1)
- P2 pad 1: (no net) -> Net-(C6-Pad1)
- P2 pad 2: /SWDIO -> GND
Routing:
- net +3V3: track 38.9 -> 0.00 mm
- net GND: track 6.64 -> 0.00 mm
- net +5V: track 2.87 -> 0.00 mm
Other:
- board outline added: 145 x 130 mm
